File: circuit/shademaker/shademaker.kicad_pcb (KiCad board)
At the start: 2 copper layers, 67.9 x 43.8 mm, 15 parts, among them M1 Jumper_NO_Small, M2 Jumper_NO_Small, Q1 IRLZ44N, SW1 I²C ADDRESS

Commit message: Circuit + PCB
Routing:
- net STEPPER_EN: track 77.8 -> 74.3 mm
Changed lines of the file:
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@@
     (thickness 1.6)
     (drawings 23)
-    (tracks 154)
+    (tracks 153)
     (zones 0)
     (modules 15)
@@
   (segment (start 168.130001 85.595001) (end 168.130001 116.695001) (width 0.25) (layer F.Cu) (net 16))
   (segment (start 165.212 82.677) (end 168.130001 85.595001) (width 0.25) (layer F.Cu) (net 16) (status 10))
-  (segment (start 173.355 116.84) (end 172.085 118.11) (width 0.25) (layer F.Cu) (net 17))
-  (segment (start 175.020002 116.84) (end 173.355 116.84) (width 0.25) (layer F.Cu) (net 17))
-  (segment (start 175.895 117.714998) (end 175.020002 116.84) (width 0.25) (layer F.Cu) (net 17))
+  (segment (start 126.365 100.965) (end 124.46 102.87) (width 0.25) (layer F.Cu) (net 17))
+  (segment (start 173.228 120.65) (end 174.244 120.65) (width 0.25) (layer F.Cu) (net 17))
+  (segment (start 124.46 102.87) (end 124.46 119.25441) (width 0.25) (layer F.Cu) (net 17))
+  (segment (start 124.46 119.25441) (end 125.85559 120.65) (width 0.25) (layer F.Cu) (net 17))
+  (segment (start 125.85559 120.65) (end 173.228 120.65) (width 0.25) (layer F.Cu) (net 17))
   (segment (start 175.895 118.999) (end 175.895 117.714998) (width 0.25) (layer F.Cu) (net 17))
   (segment (start 174.244 120.65) (end 175.895 118.999) (width 0.25) (layer F.Cu) (net 17))
-  (segment (start 125.85559 120.65) (end 174.244 120.65) (width 0.25) (layer F.Cu) (net 17))
-  (segment (start 126.365 100.965) (end 124.46 102.87) (width 0.25) (layer F.Cu) (net 17))
-  (segment (start 124.46 102.87) (end 124.46 119.25441) (width 0.25) (layer F.Cu) (net 17))
-  (segment (start 124.46 119.25441) (end 125.85559 120.65) (width 0.25) (layer F.Cu) (net 17))
+  (segment (start 175.895 117.714998) (end 175.020002 116.84) (width 0.25) (layer F.Cu) (net 17))
   (segment (start 126.615003 114.790001) (end 129.3368 117.511798) (width 0.25) (layer F.Cu) (net 18) (status 20))
   (segment (start 125.824999 114.790001) (end 126.615003 114.790001) (width 0.25) (layer F.Cu) (net 18))
