File: circuit/shademaker/shademaker.sch (KiCad schematic (older format))
At the start: 13 parts, among them M1 Jumper_NO_Small, M2 Jumper_NO_Small, Q1 IRLZ44N, SW1 I²C ADDRESS

Commit message: Circuit + PCB
Parts:
- RJ45: value 8P8C -> BLIND
Changed lines of the file:
@@
 P 10150 2350
 F 0 "RJ45" H 9820 2354 50  0000 R CNN
-F 1 "8P8C" H 9820 2445 50  0000 R CNN
+F 1 "BLIND" H 9820 2445 50  0000 R CNN
 F 2 "Connector_RJ:RJ45_Amphenol_54602-x08_Horizontal" V 10150 2375 50  0001 C CNN
 F 3 "~" V 10150 2375 50  0001 C CNN
