File: circuit/shademaker.sch (KiCad schematic (older format))
At the start: 13 parts, among them M1 Jumper_NO_Small, M2 Jumper_NO_Small, Q1 IRLZ44N, SW1 I²C ADDRESS

Commit message: Cleanup
Parts:
- RJ45: value 8P8C -> BLIND
- SCREW1: footprint TerminalBlock_RND:TerminalBlock_RND_205-00019_1x09_P5.00mm_Horizontal -> TerminalBlock_Phoenix:TerminalBlock_Phoenix_PT-1,5-9-3.5-H_1x09_P3.50mm_Horizontal
Changed lines of the file:
@@
 P 10150 2350
 F 0 "RJ45" H 9820 2354 50  0000 R CNN
-F 1 "8P8C" H 9820 2445 50  0000 R CNN
+F 1 "BLIND" H 9820 2445 50  0000 R CNN
 F 2 "Connector_RJ:RJ45_Amphenol_54602-x08_Horizontal" V 10150 2375 50  0001 C CNN
 F 3 "~" V 10150 2375 50  0001 C CNN
@@
 F 0 "SCREW1" H 10130 4292 50  0001 L CNN
 F 1 "SCREW TERMINALS" H 10130 4201 50  0000 L CNN
-F 2 "TerminalBlock_RND:TerminalBlock_RND_205-00019_1x09_P5.00mm_Horizontal" H 10050 4300 50  0001 C CNN
+F 2 "TerminalBlock_Phoenix:TerminalBlock_Phoenix_PT-1,5-9-3.5-H_1x09_P3.50mm_Horizontal" H 10050 4300 50  0001 C CNN
 F 3 "~" H 10050 4300 50  0001 C CNN
 	1    10050 4300
